Commit message: ADD CHINESE README AND USE RELATIVE PATHS THROUGHOUT
translate the readme into chinese and replace every machine-specific
absolute path with a portable relative or package:// path.

新增
---
- README_zh.md: chinese translation of the project readme
- src/mj_sim/models/meshes/: four model meshes copied next to cubot.xml
  so the mjcf can reference them with relative paths

修改
---
- README.md: link to the chinese translation and list the new meshes dir
- src/cubot_description/cubot_urdf/urdf/phantomx_urdf.xacro: use package://
  instead of the ros1 file://$(find ...) mesh uri
- src/cubot_description/cubot_urdf/urdf/cubot.urdf: replace absolute mesh
  uris with package:// and the absolute xacro source comment with a
  relative one
- src/cubot_description/cubot_urdf/urdf/wheel.xacro.bak: use package://
- src/mj_sim/models/cubot.xml: reference meshes via relative meshes/ paths
- src/mj_sim/scripts/convert_urdf.py: copy meshes next to the output and
  emit relative mesh paths
- .vscode/settings.json: use ${workspaceFolder} instead of an absolute path

File: src/cubot_description/cubot_urdf/urdf/cubot.urdf (robot description, URDF)
Before this commit: robot PhantomX, 30 links, 29 joints
Links:
- link MP_BODY: geometry collision box size=0.124 0.118 0.016; visual mesh filename=package://cubot_description/cubot_urdf/meshes/body.STL scale=1 1 1
- link c1_lf: geometry collision box size=0.026 0.022 0.01; visual mesh filename=package://cubot_description/cubot_urdf/meshes/connect.STL scale=1 1 1
- link c1_lm: geometry collision box size=0.026 0.022 0.01; visual mesh filename=package://cubot_description/cubot_urdf/meshes/connect.STL scale=1 1 1
- link c1_lr: geometry collision box size=0.026 0.022 0.01; visual mesh filename=package://cubot_description/cubot_urdf/meshes/connect.STL scale=1 1 1
- link c1_rf: geometry collision box size=0.026 0.022 0.01; visual mesh filename=package://cubot_description/cubot_urdf/meshes/connect.STL scale=1 1 1
- link c1_rm: geometry collision box size=0.026 0.022 0.01; visual mesh filename=package://cubot_description/cubot_urdf/meshes/connect.STL scale=1 1 1
- link c1_rr: geometry collision box size=0.026 0.022 0.01; visual mesh filename=package://cubot_description/cubot_urdf/meshes/connect.STL scale=1 1 1
- link c2_lf: geometry collision box size=0.026 0.022 0.01; visual mesh filename=package://cubot_description/cubot_urdf/meshes/connect.STL scale=1 1 1
- link c2_lm: geometry collision box size=0.026 0.022 0.01; visual mesh filename=package://cubot_description/cubot_urdf/meshes/connect.STL scale=1 1 1
- link c2_lr: geometry collision box size=0.026 0.022 0.01; visual mesh filename=package://cubot_description/cubot_urdf/meshes/connect.STL scale=1 1 1
- link c2_rf: geometry collision box size=0.026 0.022 0.01; visual mesh filename=package://cubot_description/cubot_urdf/meshes/connect.STL scale=1 1 1
- link c2_rm: geometry collision box size=0.026 0.022 0.01; visual mesh filename=package://cubot_description/cubot_urdf/meshes/connect.STL scale=1 1 1
- link c2_rr: geometry collision box size=0.026 0.022 0.01; visual mesh filename=package://cubot_description/cubot_urdf/meshes/connect.STL scale=1 1 1
- link thigh_lf: geometry collision box size=0.012 0.034 0.01; visual mesh filename=package://cubot_description/cubot_urdf/meshes/thigh_l.STL scale=1 1 1
- link thigh_lm: geometry collision box size=0.012 0.034 0.01; visual mesh filename=package://cubot_description/cubot_urdf/meshes/thigh_l.STL scale=1 1 1
- link thigh_lr: geometry collision box size=0.012 0.034 0.01; visual mesh filename=package://cubot_description/cubot_urdf/meshes/thigh_l.STL scale=1 1 1
- link thigh_rf: geometry collision box size=0.012 0.034 0.01; visual mesh filename=package://cubot_description/cubot_urdf/meshes/thigh_l.STL scale=1 1 1
- link thigh_rm: geometry collision box size=0.012 0.034 0.01; visual mesh filename=package://cubot_description/cubot_urdf/meshes/thigh_l.STL scale=1 1 1
- link thigh_rr: geometry collision box size=0.012 0.034 0.01; visual mesh filename=package://cubot_description/cubot_urdf/meshes/thigh_l.STL scale=1 1 1
- link tibia_lf: geometry collision box size=0.01 0.08 0.014; visual mesh filename=package://cubot_description/cubot_urdf/meshes/tibia_l.STL scale=1 1 1
- link tibia_lm: geometry collision box size=0.01 0.08 0.014; visual mesh filename=package://cubot_description/cubot_urdf/meshes/tibia_l.STL scale=1 1 1
- link tibia_lr: geometry collision box size=0.01 0.08 0.014; visual mesh filename=package://cubot_description/cubot_urdf/meshes/tibia_l.STL scale=1 1 1
- link tibia_rf: geometry collision box size=0.01 0.08 0.014; visual mesh filename=package://cubot_description/cubot_urdf/meshes/tibia_l.STL scale=1 1 1
- link tibia_rm: geometry collision box size=0.01 0.08 0.014; visual mesh filename=package://cubot_description/cubot_urdf/meshes/tibia_l.STL scale=1 1 1
- link tibia_rr: geometry collision box size=0.01 0.08 0.014; visual mesh filename=package://cubot_description/cubot_urdf/meshes/tibia_l.STL scale=1 1 1

File: src/cubot_description/cubot_urdf/urdf/phantomx_urdf.xacro (robot description, xacro)
@@ -70,5 +70,5 @@
       <origin xyz="0 0 0" rpy="0 0 0" />
       <geometry>
-        <mesh filename="file://$(find cubot_description)/cubot_urdf/meshes/body.STL" scale="1 1 1"/>
+        <mesh filename="package://cubot_description/cubot_urdf/meshes/body.STL" scale="1 1 1"/>
       </geometry>
       <material name="Grey">
@@ -111,5 +111,5 @@
       <origin xyz="0 -0.0252 0" rpy="0 0 0" />
       <geometry>
-        <mesh filename="file://$(find cubot_description)/cubot_urdf/meshes/connect.STL" scale="1 1 1"/>
+        <mesh filename="package://cubot_description/cubot_urdf/meshes/connect.STL" scale="1 1 1"/>
       </geometry>
       <material name="Grey">
@@ -137,5 +137,5 @@
       <origin xyz="0 -0.0252 0" rpy="0 0 0" />
       <geometry>
-        <mesh filename="file://$(find cubot_description)/cubot_urdf/meshes/connect.STL" scale="1 1 1"/>
+        <mesh filename="package://cubot_description/cubot_urdf/meshes/connect.STL" scale="1 1 1"/>
       </geometry>
       <material name="Grey">
@@ -164,5 +164,5 @@
       <origin xyz="0 0 0" rpy="0 0 0" />
       <geometry>
-        <mesh filename="file://$(find cubot_description)/cubot_urdf/meshes/thigh_l.STL" scale="1 1 1"/>
+        <mesh filename="package://cubot_description/cubot_urdf/meshes/thigh_l.STL" scale="1 1 1"/>
       </geometry>
       <material name="Grey">
@@ -191,5 +191,5 @@
       <origin xyz="0 0 0" rpy="0 0 0" />
       <geometry>
-        <mesh filename="file://$(find cubot_description)/cubot_urdf/meshes/tibia_l.STL" scale="1 1 1"/>
+        <mesh filename="package://cubot_description/cubot_urdf/meshes/tibia_l.STL" scale="1 1 1"/>
       </geometry>
       <material name="Grey">
